File: Board/ioWatch/ioWatch.kicad_pcb (KiCad board)
At the start: 2 copper layers, 28 x 28 mm, 85 parts, among them J1 Debug, SW1 SW_Push, SW2 SW_Push, U1 LSM6DS0, U2 STM32L031G6Ux, Y1 ABS05-32.768KHZ-T

Commit message: work
Parts:
- moved G*** 5.30 mm to (95.0, 106.8)
Routing:
- net /N1: track 0.00 -> 105.9 mm, vias 0 -> 12
- net /N2: track 0.00 -> 96.6 mm, vias 0 -> 11
- net /N3: track 0.00 -> 93.5 mm, vias 0 -> 9
- net /N4: track 0.00 -> 88.6 mm, vias 0 -> 8
- net /N5: track 0.00 -> 86.9 mm, vias 0 -> 6
- net /N6: track 0.00 -> 74.7 mm, vias 0 -> 7
- net /N8: track 0.00 -> 70.2 mm, vias 0 -> 5
- net /N7: track 0.00 -> 69.6 mm, vias 0 -> 6
- net /N9: track 0.00 -> 50.6 mm, vias 0 -> 2
- net +3.3V: track 9.00 -> 56.9 mm, vias 1 -> 6
- net GND: track 13.1 -> 53.8 mm, vias 5 -> 10
- net Net-(U2-PB7): track 0.00 -> 17.1 mm, vias 0 -> 4
- net Net-(U2-PB6): track 0.00 -> 8.99 mm, vias 0 -> 3
- added copper zone on B.Cu, net (none)
- added copper zone on F.Cu, net (none)
